Commit message: urdf update + motion trajectories

File: examples/S2full.urdf (robot description, URDF)
Before this commit: robot S2, 68 links, 67 joints
Joints:
- removed joint elbow_yaw_l_joint
- removed joint elbow_yaw_r_rjoint
- added joint wrist_yaw_l_joint: type revolute, parent elbow_pitch_l_link, child elbow_yaw_l_link, origin xyz=-0.02 0 -0.0543 rpy=0 0 0, axis 0 0 1, limit lower=-2.9670597283903604 upper=2.9670597283903604 effort=24.0 velocity=10.471975511965978
- added joint wrist_yaw_r_rjoint: type revolute, parent elbow_pitch_r_link, child elbow_yaw_r_link, origin xyz=-0.02 0 -0.0543 rpy=0 0 0, axis 0 0 1, limit lower=-2.9670597283903604 upper=2.9670597283903604 effort=24.0 velocity=10.471975511965978
- joint body_yaw_rjoint: limit lower=-2.9670597283903604 upper=3.141592653589793 effort=91.0 velocity=9.215338450530059 -> lower=-2.9670597283903604 upper=2.9670597283903604 effort=91.0 velocity=9.215338450530059
- joint shoulder_roll_l_joint: limit lower=-1.0471975511965976 upper=1.8325957145940461 effort=95.0 velocity=3.979350694547071 -> lower=-0.261799388 upper=2.61799388 effort=95.0 velocity=3.979350694547071
- joint shoulder_roll_r_rjoint: limit lower=-1.8325957145940461 upper=1.0471975511965976 effort=95.0 velocity=3.979350694547071 -> lower=-2.61799388 upper=0.261799388 effort=95.0 velocity=3.979350694547071
- joint wrist_pitch_l_joint: limit lower=-1.3089969389957472 upper=1.6580627893946132 effort=6.3 velocity=7.5398223686155035 -> lower=-0.785398163 upper=1.04719755 effort=6.3 velocity=7.5398223686155035
- joint wrist_pitch_r_rjoint: limit lower=-1.3089969389957472 upper=1.6580627893946132 effort=6.3 velocity=7.5398223686155035 -> lower=-0.785398163 upper=1.04719755 effort=6.3 velocity=7.5398223686155035
- joint wrist_roll_l_joint: limit lower=-1.0471975511965976 upper=0.7853981633974483 effort=6.3 velocity=7.5398223686155035 -> lower=-1.65806279 upper=1.30899694 effort=6.3 velocity=7.5398223686155035
- joint wrist_roll_r_rjoint: limit lower=-0.7853981633974483 upper=1.0471975511965976 effort=6.3 velocity=7.5398223686155035 -> lower=-1.30899694 upper=1.65806279 effort=6.3 velocity=7.5398223686155035

File: examples/_S2full_pybullet.urdf (robot description, URDF)
Before this commit: robot S2, 68 links, 67 joints
Joints:
- removed joint elbow_yaw_l_joint
- removed joint elbow_yaw_r_rjoint
- added joint wrist_yaw_l_joint: type revolute, parent elbow_pitch_l_link, child elbow_yaw_l_link, origin xyz=-0.02 0 -0.0543 rpy=0 0 0, axis 0 0 1, limit lower=-2.9670597283903604 upper=2.9670597283903604 effort=24.0 velocity=10.471975511965978
- added joint wrist_yaw_r_rjoint: type revolute, parent elbow_pitch_r_link, child elbow_yaw_r_link, origin xyz=-0.02 0 -0.0543 rpy=0 0 0, axis 0 0 1, limit lower=-2.9670597283903604 upper=2.9670597283903604 effort=24.0 velocity=10.471975511965978
- joint body_yaw_rjoint: limit lower=-2.9670597283903604 upper=3.141592653589793 effort=91.0 velocity=9.215338450530059 -> lower=-2.9670597283903604 upper=2.9670597283903604 effort=91.0 velocity=9.215338450530059
- joint shoulder_roll_l_joint: limit lower=-1.0471975511965976 upper=1.8325957145940461 effort=95.0 velocity=3.979350694547071 -> lower=-0.261799388 upper=2.61799388 effort=95.0 velocity=3.979350694547071
- joint shoulder_roll_r_rjoint: limit lower=-1.8325957145940461 upper=1.0471975511965976 effort=95.0 velocity=3.979350694547071 -> lower=-2.61799388 upper=0.261799388 effort=95.0 velocity=3.979350694547071
- joint wrist_pitch_l_joint: limit lower=-1.3089969389957472 upper=1.6580627893946132 effort=6.3 velocity=7.5398223686155035 -> lower=-0.785398163 upper=1.04719755 effort=6.3 velocity=7.5398223686155035
- joint wrist_pitch_r_rjoint: limit lower=-1.3089969389957472 upper=1.6580627893946132 effort=6.3 velocity=7.5398223686155035 -> lower=-0.785398163 upper=1.04719755 effort=6.3 velocity=7.5398223686155035
- joint wrist_roll_l_joint: limit lower=-1.0471975511965976 upper=0.7853981633974483 effort=6.3 velocity=7.5398223686155035 -> lower=-1.65806279 upper=1.30899694 effort=6.3 velocity=7.5398223686155035
- joint wrist_roll_r_rjoint: limit lower=-0.7853981633974483 upper=1.0471975511965976 effort=6.3 velocity=7.5398223686155035 -> lower=-1.30899694 upper=1.65806279 effort=6.3 velocity=7.5398223686155035

Commit message: dual hand inverse kimenatics, urdf updated

File: examples/S2full.urdf (robot description, URDF)
Before this commit: robot S2, 68 links, 67 joints
Links:
- added link endeffectol, mass 0.001; visual sphere radius=0.005
Joints:
- added joint endeffectol_joint: type fixed, parent L_base_link, child endeffectol, origin xyz=0.05 0.0 0.1 rpy=1.57 -1.57 -1.57

File: examples/_S2full_pybullet.urdf (robot description, URDF)
Before this commit: robot S2, 68 links, 67 joints
Links:
- added link endeffectol, mass 0.001; visual sphere radius=0.005
Joints:
- added joint endeffectol_joint: type fixed, parent L_base_link, child endeffectol, origin xyz=0.05 0.0 0.1 rpy=1.57 -1.57 -1.57

Commit message: IK for all effectors - WIP saved trajectories

File: examples/S2full.urdf (robot description, URDF)
Before this commit: robot S2, 69 links, 68 joints
Links:
- added link endeffectoh, mass 0.001; visual sphere radius=0.005
- added link endeffectoll, mass 0.001; visual sphere radius=0.005
- added link endeffectorl, mass 0.001; visual sphere radius=0.005
Joints:
- added joint endeffectoh_joint: type fixed, parent head_roll_link, child endeffectoh, origin xyz=0.2 0.0 -0.1 rpy=1.57 -1.57 -1.57
- added joint endeffectoll_joint: type fixed, parent ankle_roll_l_link, child endeffectoll, origin xyz=0.0 0.0 -0.1 rpy=1.57 -1.57 -1.57
- added joint endeffectorl_joint: type fixed, parent ankle_roll_r_link, child endeffectorl, origin xyz=0.0 0.0 -0.1 rpy=1.57 -1.57 -1.57

File: examples/_S2full_pybullet.urdf (robot description, URDF)
Before this commit: robot S2, 69 links, 68 joints
Links:
- added link endeffectoh, mass 0.001; visual sphere radius=0.005
- added link endeffectoll, mass 0.001; visual sphere radius=0.005
- added link endeffectorl, mass 0.001; visual sphere radius=0.005
Joints:
- added joint endeffectoh_joint: type fixed, parent head_roll_link, child endeffectoh, origin xyz=0.2 0.0 -0.1 rpy=1.57 -1.57 -1.57
- added joint endeffectoll_joint: type fixed, parent ankle_roll_l_link, child endeffectoll, origin xyz=0.0 0.0 -0.1 rpy=1.57 -1.57 -1.57
- added joint endeffectorl_joint: type fixed, parent ankle_roll_r_link, child endeffectorl, origin xyz=0.0 0.0 -0.1 rpy=1.57 -1.57 -1.57
